File: hardware/RaspberryPIZero-small/RaspberryPIZero-small.kicad_sch (KiCad schematic)
At the start: 29 parts, among them J1 RCVRY, J2 JTAG, J3 LPC, SW1 CPLD, SW2 BIOS

Commit message: added tooling holes to pcb & create JLCPCB manufacturing files
Parts:
- C1, C2, C3: LCSC# (none) -> C15008; MFR# (none) -> CL31A107MQHNNNE
- C4, C5: LCSC# (none) -> C14663; MFR# (none) -> CC0603KRX7R9BB104
- D1: LCSC# (none) -> C434420; MFR# (none) -> SZYY0603G
- D2: LCSC# (none) -> C434425; MFR# (none) -> SZYY0603O
- D3: LCSC# (none) -> C434419; MFR# (none) -> SZYY0603R
- D4, D5: LCSC# (none) -> C434421; MFR# (none) -> SZYY0603B
- D6: value BUSY -> CPLD; LCSC# (none) -> C434425; MFR# (none) -> SZYY0603O
- D7: value ERR -> BIOS; LCSC# (none) -> C434425; MFR# (none) -> SZYY0603O
- J2: LCSC# (none) -> C2337; MFR# (none) -> C2337
- J3: LCSC# (none) -> C57369; MFR# (none) -> C57369
- R1, R10, R11, R2, R3, R4, R5: LCSC# (none) -> C8218; MFR# (none) -> 0603WAF2000T5E
- R6, R7, R8, R9: LCSC# (none) -> C25804; MFR# (none) -> 0603WAF1002T5E
- RPI_ZERO1: LCSC# (none) -> C718226; MFR# (none) -> X6521FV-2x10-C85D32
- SW1, SW2: LCSC# (none) -> C221883; MFR# (none) -> PTS645SM70SMTR92LFS

Commit message: modified board to support flashing 49LF002A
Parts:
- added U1: SST49LF002A, 0-myparts:PLCC-32-SOCKET-SMT, symbol 0-myparts:SST49LF002A
Connections:
- net +3V3: now also U1.25 (VDD), U1.32 (VDD), U1.7 (A5/~{WP}), U1.8 (A4/~{TBL})
- net GND: now also U1.10 (A2/ID2), U1.11 (A1/ID1), U1.12 (A0/ID0), U1.16 (VSS), U1.28 (VSS), U1.29 (~{IC}/~{IC}), U1.3 (A9/FGPI3), U1.30 (A10/FPGI4), U1.4 (A8/FGPI2), U1.5 (A7/FGPI1), U1.6 (A6/FGPI0), U1.9 (A3/ID3)
- net LAD0: now also U1.13 (DQ0/FWH0)
- net LAD1: now also U1.14 (DQ1/FWH1)
- net LAD2: now also U1.15 (DQ2/FWH2)
- net LAD3: now also U1.17 (DQ3/FWH3)
- net LCLK: now also U1.31 (~{R/C}/CLK)
- net LFRAME: now also U1.23 (~{WE}/FWH4)
- net LPC_RST: now also U1.2 (~{RST})
- net ~{INIT}: now reaches RPI_ZERO1.18 (GEN5/GPIO24)
- net ~{INIT}: now also U1.24 (~{OE}/~{INIT})
Other:
- note added: "PLCC32 Socket"
